File: PCB/mysterium-pcb.kicad_sch (KiCad schematic)
At the start: 221 parts, among them J1 AVR-ISP-6, J2 OLED, J3 TRRS1, J4 TRRS2, SW0 KEYSW, SW1 KEYSW, SW10 KEYSW, SW100 KEYSW, SW101 KEYSW, SW102 KEYSW, SW103 Rotary_Encoder_Switch, SW11 KEYSW, SW12 KEYSW, SW13 KEYSW, SW14 KEYSW, SW15 KEYSW, SW16 KEYSW, SW17 KEYSW, SW18 KEYSW, SW19 KEYSW, SW2 KEYSW, SW20 KEYSW, SW21 KEYSW, SW22 KEYSW, SW23 KEYSW, SW24 KEYSW, SW25 KEYSW, SW26 KEYSW, SW27 KEYSW, SW28 KEYSW, SW29 KEYSW, SW3 KEYSW, SW30 KEYSW, SW31 KEYSW, SW32 KEYSW, SW33 KEYSW, SW34 KEYSW, SW35 KEYSW, SW36 KEYSW, SW37 KEYSW, SW38 KEYSW, SW39 KEYSW, SW4 KEYSW, SW40 KEYSW, SW41 KEYSW, SW42 KEYSW, SW43 KEYSW, SW44 KEYSW, SW45 KEYSW, SW46 KEYSW, SW47 KEYSW, SW48 KEYSW, SW49 KEYSW, SW5 KEYSW, SW50 KEYSW, SW51 KEYSW, SW52 KEYSW, SW53 KEYSW, SW54 KEYSW, SW55 KEYSW, SW56 KEYSW, SW57 KEYSW, SW58 KEYSW, SW59 KEYSW, SW6 KEYSW, SW60 KEYSW, SW61 KEYSW, SW62 KEYSW, SW63 KEYSW, SW64 KEYSW, SW65 KEYSW, SW66 KEYSW, SW67 KEYSW, SW68 KEYSW, SW69 KEYSW, SW7 KEYSW, SW70 KEYSW, SW71 KEYSW, SW72 KEYSW, SW73 KEYSW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

Commit message: Drawing columns tracks
Parts:
- SW46: now not fitted; now left out of the parts list
- SW63, SW64: now not fitted
Connections:
- net col6: now also SW83.2; no longer SW83.1
- net at D83.2 (A), SW84.2: now also SW83.1; no longer SW83.2
Changed lines of the file:
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@@
 		(lib_id "mysterium-pcb-rescue:KEYSW-keyboard_parts")
 		(at 170.18 104.14 0)
+		(mirror y)
 		(unit 1)
 		(exclude_from_sim no)
@@
 		(in_bom yes)
 		(on_board no)
-		(dnp no)
+		(dnp yes)
 		(property "Reference" "SW64"
 			(at 44.45 82.9818 0)
@@
 		(unit 1)
 		(exclude_from_sim no)
-		(in_bom yes)
-		(on_board yes)
-		(dnp no)
+		(in_bom no)
+		(on_board no)
+		(dnp yes)
 		(property "Reference" "SW46"
 			(at 311.15 52.5018 0)
@@
 		(at 311.15 73.66 0)
 		(unit 1)
-		(exclude_from_sim no)
+		(exclude_from_sim yes)
 		(in_bom yes)
-		(on_board yes)
-		(dnp no)
+		(on_board no)
+		(dnp yes)
 		(property "Reference" "SW63"
 			(at 311.15 67.7418 0)

Commit message: Finish row and columns tracks
Parts:
- SW83: footprint acheron_MXH_MetalRings:MX100H -> acheron_MXH_MetalRings:MX625HR
- SW84: footprint acheron_MXH_MetalRings:MX100H -> acheron_MXH_MetalRings:MX700HR
Changed lines of the file:
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@@
 			)
 		)
-		(property "Footprint" "acheron_MXH_MetalRings:MX100H"
+		(property "Footprint" "acheron_MXH_MetalRings:MX625HR"
 			(at 170.18 104.14 0)
 			(effects
@@
 			)
 		)
-		(property "Footprint" "acheron_MXH_MetalRings:MX100H"
+		(property "Footprint" "acheron_MXH_MetalRings:MX700HR"
 			(at 166.37 119.38 0)
 			(effects
